File: MTE_WFG-FC.kicad_pcb (KiCad board)
At the start: 2 copper layers, 200 x 75 mm, 302 parts, among them J101 Conn_02x10_Odd_Even, J102 CONN_COAXIAL, J103 CONN_COAXIAL, J104 CONN_COAXIAL, J105 CONN_COAXIAL, J106 MOLEX_KK-254, J107 MOLEX_KK-254, J108 MOLEX_KK-254, J501 Conn_01x03, J502 Conn_01x03, J503 Conn_01x04, Q201 BCW60, Q202 BCW60, Q203 BCW60, Q204 BCW60, Q205 BCW60, Q206 BCW60, Q207 BCW60, Q208 BCW60, Q601 BSS315P, Q602 BSS316N, U201 74LVC2G14, U202 74LVC273, U203 74LVC1G157, U204 AD8611, U205 AD8065, U206 74LVC1T45, U207 74LVC1G157, U208 74LVC2G14, U209 TLV1117-ADJ, U210 74LVC273, U211 AD8611, U301 AD9834, U302 MCP41050, U401 AD5721, U402 MCP9700T-E/TT, U403 LM4132-2, U404 MCP41050, U405 LM321, U406 MCP41050, U407 TLV271, U408 TLV271, U409 LM7121, U410 LMH6321, U411 AD603, U412 AD5721, U501 LM4132-2, U502 24LC04, U503 PCF8574, U504 74LVC1G157, U505 74HC138, U506 SN65MLVD203, U507 STM32F101RCTx, U508 SN65LVDS2, U509 74LVC1G157, U510 TLV1117-ADJ, U511 SN65MLVD200A, U601 TLV1117-ADJ, U602 74LVC1T45, U603 TLV271, U604 MCP9700T-E/TT, X201 FOX924B-10.000, X301 CFPS-73, Y501 16MHz

Commit message: Autosaving...
Parts:
- JP504, JP506, JP513: moved to B.Cu
- U501: value LM4132-2 -> LM4132-3.3
- moved C201 153.2 mm to (223.5, 101.0), turned to 90 degrees
- moved U202 144.4 mm to (219.0, 101.0), turned to 270 degrees
- moved C205 143.2 mm to (225.2, 102.8), turned to 270 degrees
- moved U206 142.6 mm to (228.0, 101.0), turned to 90 degrees
- moved C204 138.7 mm to (225.2, 99.2), turned to 90 degrees
- moved U201 134.1 mm to (213.8, 101.0), turned to 90 degrees
- moved C210 132.4 mm to (213.8, 96.8), turned to 90 degrees
- moved U203 128.3 mm to (210.8, 101.0), turned to 90 degrees
- moved C211 126.5 mm to (210.8, 96.8), turned to 90 degrees
- moved R207 123.6 mm to (209.2, 96.8), turned to 270 degrees
- moved J501 103.0 mm to (235.9, 55.9), turned to 0 degrees
- moved C610 89.1 mm to (47.5, 53.5)
- moved U604 83.2 mm to (51.0, 53.5), turned to 0 degrees
- moved R610 71.0 mm to (77.7, 49.5), turned to 270 degrees
- moved R612 70.3 mm to (78.5, 46.8), turned to 0 degrees
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Connections:
- C201 pad 2: GND -> DGND
- C202 pad 1: GNDA -> AGND
- C203 pad 2: GNDA -> AGND
- C204 pad 1: GND -> DGND
- C205 pad 1: GND -> DGND
- C207 pad 2: GNDA -> AGND
- C208 pad 2: GND -> DGND
- C209 pad 2: GND -> DGND
- C210 pad 2: GND -> DGND
- C211 pad 2: GND -> DGND
- C212 pad 1: GND -> DGND
- C213 pad 1: GNDA -> AGND
- C216 pad 2: GNDA -> AGND
- C217 pad 2: GNDA -> AGND
- C218 pad 1: GNDA -> AGND
- C219 pad 2: GND -> DGND
- C301 pad 2: GNDA -> AGND
- C302 pad 2: GNDA -> AGND
- C303 pad 2: GND -> DGND
- C304 pad 2: GNDA -> AGND
- C305 pad 2: GND -> DGND
- C310 pad 2: GNDA -> AGND
- C315 pad 2: GND -> DGND
- C319 pad 2: GND -> DGND
- C401 pad 2: GND -> DGND
- C402 pad 2: GNDA -> AGND
- C403 pad 1: GNDA -> AGND
- C404 pad 2: GNDA -> AGND
- C405 pad 2: GNDA -> AGND
- C406 pad 1: GNDA -> AGND
- C407 pad 1: GNDA -> AGND
- C408 pad 2: GND -> DGND
- C409 pad 2: GNDA -> AGND
- C410 pad 1: GND -> DGND
- C411 pad 1: GNDA -> AGND
- C412 pad 1: GNDA -> AGND
- C413 pad 1: GNDA -> AGND
- C414 pad 2: GNDA -> AGND
- C415 pad 2: GNDA -> AGND
- C416 pad 1: GNDA -> AGND
- C417 pad 2: GNDA -> AGND
- C418 pad 1: GNDA -> AGND
- C419 pad 2: GNDA -> AGND
- C422 pad 2: GNDA -> AGND
- C423 pad 1: GNDA -> AGND
- C424 pad 1: GNDA -> AGND
- C426 pad 2: GNDA -> AGND
- C427 pad 2: GNDA -> AGND
- C428 pad 2: GNDA -> AGND
- C429 pad 2: GNDA -> AGND
- C430 pad 2: GND -> DGND
- C431 pad 2: GNDA -> AGND
- C432 pad 2: GNDA -> AGND
- C501 pad 2: GND -> DGND
- C502 pad 1: GND -> DGND
- C503 pad 2: GNDA -> AGND
- C504 pad 1: GNDA -> AGND
- C505 pad 2: GNDA -> AGND
- C506 pad 2: GND -> DGND
- C507 pad 1: GND -> DGND
- C508 pad 2: GND -> DGND
- C509 pad 1: GND -> DGND
- C510 pad 2: GND -> DGND
- C511 pad 1: GND -> DGND
- C512 pad 2: GND -> DGND
- C513 pad 1: GND -> DGND
- C514 pad 2: GND -> DGND
- C515 pad 2: GND -> DGND
- C516 pad 2: GND -> DGND
- C517 pad 2: GND -> DGND
- C518 pad 2: GND -> DGND
- C519 pad 2: GND -> DGND
- C520 pad 2: GND -> DGND
- C521 pad 2: GND -> DGND
- C522 pad 2: GND -> DGND
- C523 pad 1: GND -> DGND
- C524 pad 2: GND -> DGND
- C601 pad 2: GND -> AGND
- C602 pad 2: GND -> DGND
- C603 pad 1: GND -> DGND
- C604 pad 1: GND -> DGND
- C605 pad 2: GND -> DGND
- C606 pad 2: GND -> DGND
- C607 pad 2: GND -> DGND
- C608 pad 1: GND -> DGND
- C609 pad 2: GND -> DGND
- C610 pad 1: GNDA -> AGND
- J101 pad 11: GND -> DGND
- J101 pad 14: GND -> DGND
- J101 pad 17: GND -> DGND
- J101 pad 2: GND -> DGND
- J101 pad 20: GND -> DGND
- J101 pad 4: GND -> DGND
- J101 pad 6: GND -> DGND
- J101 pad 8: GND -> DGND
- J102 pad 2: GNDA -> AGND
- J103 pad 2: GNDA -> AGND
- J104 pad 2: GNDA -> AGND
- J105 pad 2: GND -> DGND
- J106 pad 2: GNDA -> AGND
- J106 pad 4: GNDA -> AGND
- J106 pad 6: GNDA -> AGND
- J106 pad 8: GNDA -> AGND
- J107 pad 10: GND -> DGND
- J107 pad 12: GND -> DGND
- J107 pad 2: GND -> DGND
- J107 pad 4: GND -> DGND
- J107 pad 6: GND -> DGND
- J107 pad 8: GND -> DGND
- J108 pad 10: GND -> DGND
- J108 pad 12: GND -> DGND
- J108 pad 2: GND -> DGND
- J108 pad 4: GND -> DGND
- J108 pad 6: GND -> DGND
- J108 pad 8: GND -> DGND
- J502 pad 3: GND -> DGND
- J503 pad 4: GND -> DGND
- JP501 pad 2: GND -> DGND
- JP502 pad 2: GND -> DGND
- JP503 pad 2: GND -> DGND
- JP507 pad 2: GND -> DGND
- JP508 pad 2: GND -> DGND
- JP509 pad 2: GND -> DGND
- JP510 pad 2: GND -> DGND
- JP511 pad 2: GND -> DGND
- JP512 pad 2: GND -> DGND
- NT301 pad 1: GND -> DGND
- NT301 pad 2: GNDA -> AGND
- NT301 pad 3: GND -> DGND
- NT301 pad 4: GNDA -> AGND
- NT401 pad 1: GND -> DGND
- NT401 pad 2: GNDA -> AGND
- NT401 pad 3: GND -> DGND
- NT401 pad 4: GNDA -> AGND
- NT402 pad 1: GND -> DGND
- NT402 pad 2: GNDA -> AGND
- NT402 pad 3: GND -> DGND
- NT402 pad 4: GNDA -> AGND
- NT403 pad 1: GND -> DGND
- NT403 pad 2: GNDA -> AGND
- NT403 pad 3: GND -> DGND
- NT403 pad 4: GNDA -> AGND
- NT404 pad 1: GND -> DGND
- NT404 pad 2: GNDA -> AGND
- NT404 pad 3: GND -> DGND
- NT404 pad 4: GNDA -> AGND
- NT501 pad 1: GNDA -> AGND
- NT501 pad 2: GND -> DGND
- NT501 pad 3: GNDA -> AGND
- NT501 pad 4: GND -> DGND
- Q203 pad 3: GNDA -> AGND
- Q204 pad 1: GNDA -> AGND
- Q204 pad 2: GNDA -> AGND
- Q207 pad 3: GNDA -> AGND
- Q208 pad 1: GNDA -> AGND
- Q208 pad 2: GNDA -> AGND
- Q602 pad 3: GND -> DGND
- R207 pad 1: GND -> DGND
- R208 pad 2: GNDA -> AGND
- R211 pad 2: GNDA -> AGND
- R217 pad 2: GND -> DGND
- R218 pad 2: GNDA -> AGND
- R220 pad 2: GNDA -> AGND
- R221 pad 2: GNDA -> AGND
- R222 pad 2: GNDA -> AGND
- R302 pad 1: GNDA -> AGND
- R303 pad 2: GNDA -> AGND
- R304 pad 2: GNDA -> AGND
- R305 pad 2: GNDA -> AGND
- R306 pad 2: GNDA -> AGND
- R409 pad 1: GNDA -> AGND
- R412 pad 1: GNDA -> AGND
- R416 pad 1: GNDA -> AGND
- R428 pad 2: GNDA -> AGND
- R429 pad 2: GNDA -> AGND
- R506 pad 1: GND -> DGND
- R508 pad 1: GND -> DGND
- R511 pad 2: GND -> DGND
- R512 pad 2: GND -> DGND
- R513 pad 2: GND -> DGND
- R514 pad 2: GND -> DGND
- R517 pad 2: GND -> DGND
- R602 pad 2: GND -> AGND
- R611 pad 1: GND -> DGND
- R612 pad 1: GND -> DGND
- U201 pad 2: GND -> DGND
- U202 pad 10: GND -> DGND
- U202 pad 14: GND -> DGND
- U202 pad 17: GND -> DGND
- U202 pad 18: GND -> DGND
- U203 pad 2: GND -> DGND
- U204 pad 4: GNDA -> AGND
- U204 pad 5: GNDA -> AGND
- U204 pad 6: GNDA -> AGND
- U206 pad 2: GND -> DGND
- U206 pad 5: GND -> DGND
- U207 pad 2: GND -> DGND
- U208 pad 2: GND -> DGND
- U210 pad 10: GND -> DGND
- U210 pad 14: GND -> DGND
- U210 pad 17: GND -> DGND
- U210 pad 18: GND -> DGND
- U211 pad 4: GNDA -> AGND
- U211 pad 5: GNDA -> AGND
- U211 pad 6: GNDA -> AGND
- U301 pad 10: GND -> DGND
- U301 pad 12: GND -> DGND
- U301 pad 17: GNDA -> AGND
- U301 pad 18: GNDA -> AGND
- U301 pad 7: GND -> DGND
- U301 pad 9: GND -> DGND
- U302 pad 1: /~FS_ADJ~ -> /~ADJ_FS~
- U302 pad 4: GND -> DGND
- U401 pad 16: GND -> DGND
- U401 pad 5: GNDA -> AGND
- U402 pad 3: GNDA -> AGND
- U403 pad 2: GNDA -> AGND
- U404 pad 4: GND -> DGND
- U404 pad 7: GNDA -> AGND
- U406 pad 4: GND -> DGND
- U407 pad 2: GNDA -> AGND
- U410 pad 2: GNDA -> AGND
- U411 pad 1: GNDA -> AGND
- U411 pad 4: GNDA -> AGND
- U412 pad 16: GND -> DGND
- U412 pad 5: GNDA -> AGND
- U501 pad 2: GNDA -> AGND
- U502 pad 1: GND -> DGND
- U502 pad 2: GND -> DGND
- U502 pad 3: GND -> DGND
- U502 pad 4: GND -> DGND
- U503 pad 8: GND -> DGND
- U504 pad 5: GND -> DGND
- U505 pad 11: /~LVL_CL~ -> /~ADJ_NULL~
- U505 pad 12: /~ADJ_NULL~ -> /~ADJ_FS~
- U505 pad 13: /~DDS~ -> /~LVL_CL~
- U505 pad 14: /~FS_ADJ~ -> /~DDS~
- U505 pad 4: GND -> DGND
- U505 pad 5: GND -> DGND
- U505 pad 8: GND -> DGND
- U506 pad 6: GND -> DGND
- U506 pad 7: GND -> DGND
- U507 pad 10: /TMON0 -> (no net)
- U507 pad 11: /TMON1 -> (no net)
- U507 pad 12: GNDA -> AGND
- U507 pad 14: (no net) -> /Analog Output Stage/UMON_OUT
- U507 pad 15: (no net) -> /Analog Output Stage/FB_NULL
- U507 pad 16: /Analog Output Stage/UMON_OUT -> /UMON_VREF
- U507 pad 17: /Analog Output Stage/FB_NULL -> /UMON_SQR
- U507 pad 18: GND -> DGND
- U507 pad 20: /Control logic/ADJ_TRIG -> /ADJ_SQR
- U507 pad 21: /ADJ_SQR -> /Control logic/ADJ_TRIG
- U507 pad 22: /UMON_SQR -> /TMON0
- U507 pad 23: /UMON_VREF -> /TMON1
- U507 pad 29: /SQR -> Net-(U507-Pad29)
- U507 pad 30: Net-(U507-Pad30) -> /SQR
- U507 pad 31: GND -> DGND
- U507 pad 41: (no net) -> Net-(R508-Pad2)
- U507 pad 44: Net-(R508-Pad2) -> (no net)
- U507 pad 47: GND -> DGND
- U507 pad 63: GND -> DGND
- U508 pad 2: GND -> DGND
- U509 pad 1: Net-(U507-Pad30) -> Net-(U507-Pad29)
- U509 pad 5: GND -> DGND
- U511 pad 5: GND -> DGND
- U602 pad 2: GND -> DGND
- U602 pad 5: GND -> DGND
- U603 pad 2: GND -> DGND
- U604 pad 3: GNDA -> AGND
- X201 pad 2: GND -> DGND
- X301 pad 2: GND -> DGND
- Y501 pad 2: GND -> DGND
- Y501 pad 4: GND -> DGND
Routing:
- net +3V3D: track 45.6 -> 461.1 mm, vias 0 -> 16
- net Net-(C602-Pad1): track 0.00 -> 280.0 mm, vias 0 -> 13
- net /ADJ_SQR: track 0.00 -> 254.3 mm, vias 0 -> 4
- net /TMON0: track 0.00 -> 217.9 mm
- net +5V0A: track 30.5 -> 241.8 mm, vias 0 -> 13
- net /EF: track 0.00 -> 196.3 mm, vias 0 -> 2
- net /TMON1: track 0.00 -> 194.1 mm
- net /SIG_D: track 0.00 -> 190.8 mm
- net +3V3A: track 11.9 -> 201.2 mm
- net +5V0D: track 0.00 -> 186.8 mm, vias 0 -> 2
- net -15V: track 11.2 -> 157.6 mm, vias 2 -> 47
- net +15V: track 11.7 -> 157.4 mm, vias 2 -> 5
- net Net-(U204-Pad8): track 0.00 -> 141.5 mm
- net +12V: track 0.00 -> 138.1 mm, vias 0 -> 1
- net VREF: track 0.00 -> 136.5 mm, vias 0 -> 4
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- added copper zone on B.Cu, net -15V
- added copper zone on F.Cu, net -15V
- added copper zone on B.Cu, net AGND
- added copper zone on F.Cu, net AGND
- added copper zone on B.Cu, net DGND
- added copper zone on F.Cu, net DGND
- added copper zone on B.Cu, net Net-(C602-Pad1)
- added copper zone on F.Cu, net Net-(C602-Pad1)
